File: AKD52_Rev1.kicad_sch (KiCad schematic)
At the start: 9 parts, among them J1 DIN41612_03x32_C_Split, J2 Conn_01x02, J3 Conn_02x17_Odd_Even, J4 Conn_02x10_Odd_Even, U1 74HCT245, U2 74HCT245, U3 74HCT273, U4 PAL16L8, U5 2764

Commit message: Worked on schematic missing 26LS32
Parts:
- added J5: Conn_02x10_Odd_Even, symbol Connector_Generic:Conn_02x10_Odd_Even
- added U6: AM26LS31CN, Package_DIP:DIP-16_W7.62mm, symbol Interface:AM26LS31CN
- renumbered J1 to PL1
Other:
- moved on the sheet: J1C, J2, J3, J4, U1, U2, U3, U4, U5

Commit message: Worked on connectors for harddrive
Parts:
- added C1, C2: C, symbol Device:C
- added R13: 330, symbol Device:R
- added R14, R15: 100, symbol Device:R
- added U15, U9: 74HC14, symbol 74xx:74HC14
- added U16, U8: 74LS04, symbol 74xx:74LS04
- added U7: AM26LV32xD, Package_SO:SOIC-16_3.9x9.9mm_P1.27mm, symbol Interface:AM26LV32xD
Connections:
- net GNDD: now reaches U6.12 (~{G})
- net GNDD: now also U6.15 (4A), U6.8 (GND), U6.9 (3A), C1.2, C2.2, U7.10 (3A), U7.12 (~{G}), U7.6 (2A), U7.7 (2B), U7.8 (GND), U7.9 (3B)
- net +5VD: now reaches U6.16 (VDD)
- net +5VD: now also J2.1 (Pin_1), C1.1, C2.1, U7.16 (VDD), U7.4 (G)
- net at U6.2 (1Y): now also J4.13 (Pin_13)
- net at U6.3 (1Z): now also J4.14 (Pin_14)
- net at U6.5 (2Z): now also J5.14 (Pin_14)
- net at U6.6 (2Y): now also J5.13 (Pin_13)
- net at J2.2 (Pin_2): now also R13.2
- net at J4.17 (Pin_17): now also R14.1, U7.1 (1B)
- net at J4.18 (Pin_18): now also R14.2, U7.2 (1A)
- net at J3.12 (Pin_12): now also U15.5
- net at J3.14 (Pin_14): now also U8.6
- net at J3.18 (Pin_18): now also U8.4
- net at J3.22 (Pin_22): now also U15.1
- net at J3.26 (Pin_26): now also U16.10
- net at J3.28 (Pin_28): now also U8.8
- net at J3.4 (Pin_4): now also U8.2
- net at J3.6 (Pin_6): now also U8.12
- net at J3.8 (Pin_8): now also U15.3
- net at J5.17 (Pin_17): now also R15.1, U7.15 (4B)
- net at J5.18 (Pin_18): now also R15.2, U7.14 (4A)
Other:
- moved on the sheet: J2, J4, Reference: J3, U6
